File: electronics/hiside_switch/hiside_switch.kicad_sch (KiCad schematic)
At the start: 20 parts, among them J1 Screw_Terminal_01x02, J2 Screw_Terminal_01x02, J3 Conn_01x04_Pin, Q1 BC848, U2 BTS6163D

Commit message: routing completed
Parts:
- added C1, C6: C, Capacitor_SMD:C_0805_2012Metric_Pad1.18x1.45mm_HandSolder, symbol Device:C
- added C5: C, Capacitor_THT:C_Rect_L7.2mm_W4.5mm_P5.00mm_FKS2_FKP2_MKS2_MKP2, symbol Device:C
- added R1, R7: R, Resistor_SMD:R_0805_2012Metric_Pad1.20x1.40mm_HandSolder, symbol Device:R
- TH1: footprint Varistor:RV_Disc_D12mm_W4.5mm_P7.5mm -> Varistor:RV_Disc_D9mm_W3.3mm_P5mm
- renumbered C1 to C2, C2 to C3, C3 to C4, J3 to J1, J1 to J3, R6 to R2, R5 to R3, R3 to R5, R2 to R6, R1 to R8, U2 to U1
Connections:
- net GND: now reaches C2.2, C3.2, C4.2, D1.2 (A), J2.2 (Pin_2), J3.1 (Pin_1), Q1.2 (E), R3.1, R4.2, R5.2, R8.2
- net GND: now also J1.2 (Pin_2), C1.2, C5.2, C6.2; no longer J1.4 (Pin_4)
- net pout: now reaches J3.2 (Pin_2), U1.1 (OUT), U1.5 (OUT)
- net VCC: now reaches C2.1, C3.1, C4.1, D1.1 (K), R4.1, R5.1, TH1.1, U1.3 (Vbb)
- net VCC: now also C5.1, R1.2; no longer R2.2
- net at R2.1, R3.2: now also J1.3 (Pin_3), C1.1; no longer J1.1 (Pin_1)
- net at R6.1: now also J1.1 (Pin_1); no longer J1.2 (Pin_2)
- net at R8.1, U1.4 (IS): now also R7.2; no longer J1.3 (Pin_3)
- new net: R1.1, R2.2
- new net: C6.1, J1.4 (Pin_4), R7.1
Other:
- moved on the sheet: J1, Q1, R2, R3, R6
